File: Learn404.sch (KiCad schematic (older format))
At the start: 88 parts, among them U1 LM555, U2 4520

Commit message: Uploaded Rev B files. This board is known to work.
Parts:
- BT1, BT2: footprint Battery:3039 -> Battery:BatteryHolder_Keystone_3009_1x2450
- D1, D2, D3, D4, D5, D6, D7, D8: footprint LED_SMD:LED_1206_3216Metric -> Resistor_SMD:R_1210_3225Metric_Pad1.42x2.65mm_HandSolder
- R1, R10, R11, R12, R13, R14, R15, R16, R17, R18, R19, R2, R20, R21, R22, R23, R24, R25, R26, R27, R28, R29, R3, R30, R31, R32, R4, R5, R6, R65, R66, R67, R68, R69, R7, R70, R8, R9: footprint Resistor_THT:R_Axial_DIN0207_L6.3mm_D2.5mm_P7.62mm_Horizontal -> Resistor_THT:R_Axial_DIN0207_L6.3mm_D2.5mm_P10.16mm_Horizontal
- R33, R34, R35, R36, R37, R38, R39, R40, R41, R42, R43, R44, R45, R46, R47, R48, R49, R50, R51, R52, R53, R54, R55, R56, R57, R58, R59, R60, R61, R62, R63, R64, R71, R72, R73, R74: footprint Resistor_SMD:R_1206_3216Metric -> Resistor_SMD:R_1206_3216Metric_Pad1.42x1.75mm_HandSolder
Other:
- note added: "Cell Holder: 36-3039-ND\n1Ah Cell: 1908-1388-ND\n\nAlternate: \nCell Holder: 36-3009-ND\n580mAh Cell: 2059-CR2450-ND"
- note removed: "Cell Holder: 36-3039-ND\n1Ah Cell: 1908-1388-ND"
